Commit message: added lidar support files

File: Automation/src/lidar_sensor/urdf/lidar.xacro (robot description, xacro)
@@ -7,5 +7,5 @@
         <box size="0.3 0.3 0.1"/>
       </geometry>
-      <material>
+      <material name="mat_1">
         <color rgba="0.7 0.7 0.7 1"/>
       </material>
@@ -27,5 +27,5 @@
         <cylinder length="0.05" radius="0.03"/>
       </geometry>
-      <material>
+      <material name="mat_2">
         <color rgba="0.0 0.8 0.0 1.0"/>
       </material>
